Commit message: feat: add two links and two joints

File: src/arduinobot_description/urdf/arduinobot.urdf.xacro (robot description, xacro)
@@ -24,4 +24,20 @@
         </visual>
     </link>
+    <link name="forward_drive_arm">
+        <visual>
+            <origin rpy="0 -${PI/2} ${PI/2}"  xyz="0.19 0.06 -0.08" />
+            <geometry>
+                <mesh filename="package://arduinobot_description/meshes/forward_drive_arm.STL" scale="0.01 0.01 0.01" />
+            </geometry>
+        </visual>
+    </link>
+    <link name="horizontal_arm">
+        <visual>
+            <origin rpy="${PI/2} 0 ${PI/2}"  xyz="-0.03 -0.4 -0.06" />
+            <geometry>
+                <mesh filename="package://arduinobot_description/meshes/horizontal_arm.STL" scale="0.01 0.01 0.01" />
+            </geometry>
+        </visual>
+    </link>
     <!-- JOINTS STATE -->
     <!-- We linked two links - world with base link  -->
@@ -39,3 +55,17 @@
         <limit lower="-${PI/2}" upper="${PI/2}" effort="${effort}" velocity="${velocity}" />
     </joint>
+    <joint name="joint_2" type="revolute">
+        <parent link="base_plate" />
+        <child link="forward_drive_arm" />
+        <axis xyz="1 0 0" />
+        <origin rpy="0 0 0" xyz="-0.2 0 0.35" />
+        <limit lower="-${PI/2}" upper="${PI/2}" effort="${effort}" velocity="${velocity}" />
+    </joint>
+    <joint name="joint_3" type="revolute">
+        <parent link="forward_drive_arm" />
+        <child link="horizontal_arm" />
+        <axis xyz="1 0 0" />
+        <origin rpy="0 0 0" xyz="0 0 0.8" />
+        <limit lower="-${PI/2}" upper="${PI/2}" effort="${effort}" velocity="${velocity}" />
+    </joint>
 </robot>

Commit message: chore: change xyz

File: src/arduinobot_description/urdf/arduinobot.urdf.xacro (robot description, xacro)
@@ -34,5 +34,5 @@
     <link name="horizontal_arm">
         <visual>
-            <origin rpy="${PI/2} 0 ${PI/2}"  xyz="-0.03 -0.4 -0.06" />
+            <origin rpy="${PI/2} 0 ${PI/2}"  xyz="-0.03 -0.42 -0.081" />
             <geometry>
                 <mesh filename="package://arduinobot_description/meshes/horizontal_arm.STL" scale="0.01 0.01 0.01" />

Commit message: chore: fix xyz of the link with joint

File: src/arduinobot_description/urdf/arduinobot.urdf.xacro (robot description, xacro)
@@ -34,5 +34,5 @@
     <link name="horizontal_arm">
         <visual>
-            <origin rpy="${PI/2} 0 ${PI/2}"  xyz="-0.03 -0.42 -0.081" />
+            <origin rpy="${PI/2} 0 ${PI/2}"  xyz="-0.03 -0.425 -0.073" />
             <geometry>
                 <mesh filename="package://arduinobot_description/meshes/horizontal_arm.STL" scale="0.01 0.01 0.01" />
@@ -66,5 +66,5 @@
         <child link="horizontal_arm" />
         <axis xyz="1 0 0" />
-        <origin rpy="0 0 0" xyz="0 0 0.8" />
+        <origin rpy="0 0 0" xyz="0 0.008 0.793" />
         <limit lower="-${PI/2}" upper="${PI/2}" effort="${effort}" velocity="${velocity}" />
     </joint>

Commit message: chore: fix xyz

File: src/arduinobot_description/urdf/arduinobot.urdf.xacro (robot description, xacro)
@@ -26,5 +26,5 @@
     <link name="forward_drive_arm">
         <visual>
-            <origin rpy="0 -${PI/2} ${PI/2}"  xyz="0.19 0.06 -0.08" />
+            <origin rpy="0 -${PI/2} ${PI/2}"  xyz="0.19 0.073 -0.079" />
             <geometry>
                 <mesh filename="package://arduinobot_description/meshes/forward_drive_arm.STL" scale="0.01 0.01 0.01" />
@@ -59,5 +59,5 @@
         <child link="forward_drive_arm" />
         <axis xyz="1 0 0" />
-        <origin rpy="0 0 0" xyz="-0.2 0 0.35" />
+        <origin rpy="0 0 0" xyz="-0.2 0.022 0.354" />
         <limit lower="-${PI/2}" upper="${PI/2}" effort="${effort}" velocity="${velocity}" />
     </joint>
@@ -66,5 +66,5 @@
         <child link="horizontal_arm" />
         <axis xyz="1 0 0" />
-        <origin rpy="0 0 0" xyz="0 0.008 0.793" />
+        <origin rpy="0 0 0" xyz="0 0.02 0.793" />
         <limit lower="-${PI/2}" upper="${PI/2}" effort="${effort}" velocity="${velocity}" />
     </joint>

Commit message: feat: complete the urdf model

File: src/arduinobot_description/urdf/arduinobot.urdf.xacro (robot description, xacro)
@@ -40,4 +40,28 @@
         </visual>
     </link>
+    <link name="claw_support">
+        <visual>
+            <origin rpy="0 0 ${PI/2}"  xyz="0 -0.06 -0.15" />
+            <geometry>
+                <mesh filename="package://arduinobot_description/meshes/claw_support.STL" scale="0.01 0.01 0.01" />
+            </geometry>
+        </visual>
+    </link>
+    <link name="gripper_right">
+        <visual>
+            <origin rpy="0 0 -${PI/2}"  xyz="-0.107 0.4744 -0.1" />
+            <geometry>
+                <mesh filename="package://arduinobot_description/meshes/right_finger.STL" scale="0.01 0.01 0.01" />
+            </geometry>
+        </visual>
+    </link>
+    <link name="gripper_left">
+        <visual>
+            <origin rpy="0 0 -${PI/2}"  xyz="-0.039 0.4744 -0.1" />
+            <geometry>
+                <mesh filename="package://arduinobot_description/meshes/left_finger.STL" scale="0.01 0.01 0.01" />
+            </geometry>
+        </visual>
+    </link>
     <!-- JOINTS STATE -->
     <!-- We linked two links - world with base link  -->
@@ -69,3 +93,23 @@
         <limit lower="-${PI/2}" upper="${PI/2}" effort="${effort}" velocity="${velocity}" />
     </joint>
+    <joint name="horizontal_arm_to_claw_support" type="fixed">
+        <parent link="horizontal_arm" />
+        <child link="claw_support" />
+        <origin rpy="0 0 0" xyz="0 0.80 0" />
+    </joint>
+    <joint name="joint_4" type="revolute">
+        <parent link="claw_support" />
+        <child link="gripper_right" />
+        <axis xyz="0 0 1" />
+        <origin rpy="0 0 0" xyz="-0.035 0.147 -0.1" />
+        <limit lower="-${PI/2}" upper="0.0" effort="${effort}" velocity="${velocity}" />
+    </joint>
+    <joint name="joint_5" type="revolute">
+        <parent link="claw_support" />
+        <child link="gripper_left" />
+        <axis xyz="0 0 1" />
+        <origin rpy="0 0 0" xyz="-0.215 0.147 -0.1" />
+        <mimic joint="joint_4" multiplier="-1" />
+        <limit lower="0.0" upper="${PI/2}" effort="${effort}" velocity="${velocity}" />
+    </joint>
 </robot>

Commit message: feat: add link and joint for rgb camera

File: src/arduinobot_description/urdf/arduinobot.urdf.xacro (robot description, xacro)
@@ -9,8 +9,15 @@
     <link name="base_link">
         <visual>
-            <!-- Orientation and position only for mesh -->
             <origin rpy="0 0 0"  xyz="-0.5 -0.5 0" />
             <geometry>
                 <mesh filename="package://arduinobot_description/meshes/basement.STL" scale="0.01 0.01 0.01" />
+            </geometry>
+        </visual>
+    </link>
+    <link name="rgb_camera">
+        <visual>
+            <origin rpy="-1.1 0 0"  xyz="-0.15 0.34 0.28" />
+            <geometry>
+                <mesh filename="package://arduinobot_description/meshes/pi_camera.STL" scale="0.01 0.01 0.01" />
             </geometry>
         </visual>
@@ -64,10 +71,12 @@
         </visual>
     </link>
-    <!-- JOINTS STATE -->
-    <!-- We linked two links - world with base link  -->
     <joint name="virtual_joint" type="fixed">
         <parent link="world" />
         <child link="base_link" />
-        <!-- Orientation and position for joint  -->
+        <origin rpy="0 0 0" xyz="0 0 0" />
+    </joint>
+    <joint name="rgb_camera_joint" type="fixed">
+        <parent link="base_link" />
+        <child link="rgb_camera" />
         <origin rpy="0 0 0" xyz="0 0 0" />
     </joint>

Commit message: feat: add default_inertial to urdf links

File: src/arduinobot_description/urdf/arduinobot.urdf.xacro (robot description, xacro)
@@ -6,6 +6,13 @@
     <xacro:property name="effort" value="30.0" />
     <xacro:property name="velocity" value="10.0" />
+    <xacro:macro name="default_inertial" params="mass">
+        <inertial>
+            <mass value="${mass}" />
+            <inertia ixx="1.0" ixy="0.0" ixz="0.0" iyy="1.0" iyz="0.0" izz="1.0" />
+        </inertial>
+    </xacro:macro>
     <link name="world" />
     <link name="base_link">
+        <xacro:default_inertial mass="1.0" />
         <visual>
             <origin rpy="0 0 0"  xyz="-0.5 -0.5 0" />
@@ -14,4 +21,10 @@
             </geometry>
         </visual>
+        <collision>
+            <origin rpy="0 0 0"  xyz="-0.5 -0.5 0" />
+            <geometry>
+                <mesh filename="package://arduinobot_description/meshes/basement.STL" scale="0.01 0.01 0.01" />
+            </geometry>
+        </collision>
     </link>
     <link name="rgb_camera">
@@ -22,6 +35,13 @@
             </geometry>
         </visual>
+        <collision>
+            <origin rpy="-1.1 0 0"  xyz="-0.15 0.34 0.28" />
+            <geometry>
+                <mesh filename="package://arduinobot_description/meshes/pi_camera.STL" scale="0.01 0.01 0.01" />
+            </geometry>
+        </collision>
     </link>
     <link name="base_plate">
+        <xacro:default_inertial mass="0.1" />
         <visual>
             <origin rpy="0 0 0"  xyz="-0.39 -0.39 -0.56" />
@@ -30,6 +50,13 @@
             </geometry>
         </visual>
+        <collision>
+            <origin rpy="0 0 0"  xyz="-0.39 -0.39 -0.56" />
+            <geometry>
+                <mesh filename="package://arduinobot_description/meshes/base_plate.STL" scale="0.01 0.01 0.01" />
+            </geometry>
+        </collision>
     </link>
     <link name="forward_drive_arm">
+        <xacro:default_inertial mass="0.1" />
         <visual>
             <origin rpy="0 -${PI/2} ${PI/2}"  xyz="0.19 0.073 -0.079" />
@@ -38,6 +65,13 @@
             </geometry>
         </visual>
+        <collision>
+            <origin rpy="0 -${PI/2} ${PI/2}"  xyz="0.19 0.073 -0.079" />
+            <geometry>
+                <mesh filename="package://arduinobot_description/meshes/forward_drive_arm.STL" scale="0.01 0.01 0.01" />
+            </geometry>
+        </collision>
     </link>
     <link name="horizontal_arm">
+        <xacro:default_inertial mass="0.1" />
         <visual>
             <origin rpy="${PI/2} 0 ${PI/2}"  xyz="-0.03 -0.425 -0.073" />
@@ -46,6 +80,13 @@
             </geometry>
         </visual>
+        <collision>
+            <origin rpy="${PI/2} 0 ${PI/2}"  xyz="-0.03 -0.425 -0.073" />
+            <geometry>
+                <mesh filename="package://arduinobot_description/meshes/horizontal_arm.STL" scale="0.01 0.01 0.01" />
+            </geometry>
+        </collision>
     </link>
     <link name="claw_support">
+        <xacro:default_inertial mass="0.05" />
         <visual>
             <origin rpy="0 0 ${PI/2}"  xyz="0 -0.06 -0.15" />
@@ -54,6 +95,13 @@
             </geometry>
         </visual>
+        <collision>
+            <origin rpy="0 0 ${PI/2}"  xyz="0 -0.06 -0.15" />
+            <geometry>
+                <mesh filename="package://arduinobot_description/meshes/claw_support.STL" scale="0.01 0.01 0.01" />
+            </geometry>
+        </collision>
     </link>
     <link name="gripper_right">
+        <xacro:default_inertial mass="0.01" />
         <visual>
             <origin rpy="0 0 -${PI/2}"  xyz="-0.107 0.4744 -0.1" />
@@ -62,6 +110,13 @@
             </geometry>
         </visual>
+        <collision>
+            <origin rpy="0 0 -${PI/2}"  xyz="-0.107 0.4744 -0.1" />
+            <geometry>
+                <mesh filename="package://arduinobot_description/meshes/right_finger.STL" scale="0.01 0.01 0.01" />
+            </geometry>
+        </collision>
     </link>
     <link name="gripper_left">
+        <xacro:default_inertial mass="0.01" />
         <visual>
             <origin rpy="0 0 -${PI/2}"  xyz="-0.039 0.4744 -0.1" />
@@ -70,4 +125,10 @@
             </geometry>
         </visual>
+        <collision>
+            <origin rpy="0 0 -${PI/2}"  xyz="-0.039 0.4744 -0.1" />
+            <geometry>
+                <mesh filename="package://arduinobot_description/meshes/left_finger.STL" scale="0.01 0.01 0.01" />
+            </geometry>
+        </collision>
     </link>
     <joint name="virtual_joint" type="fixed">

Commit message: fix: urdf and launch files

File: src/arduinobot_description/urdf/arduinobot.urdf.xacro (robot description, xacro)
@@ -30,5 +30,5 @@
     <link name="rgb_camera">
         <visual>
-            <origin rpy="-1.1 0 0"  xyz="-0.15 0.34 0.28" />
+            <origin rpy="-${PI/2} 0 -${PI/2}" xyz="-0.1 0.125 0.15"/>
             <geometry>
                 <mesh filename="package://arduinobot_description/meshes/pi_camera.STL" scale="0.01 0.01 0.01" />
@@ -137,9 +137,4 @@
         <origin rpy="0 0 0" xyz="0 0 0" />
     </joint>
-    <joint name="rgb_camera_joint" type="fixed">
-        <parent link="base_link" />
-        <child link="rgb_camera" />
-        <origin rpy="0 0 0" xyz="0 0 0" />
-    </joint>
     <joint name="joint_1" type="revolute">
         <parent link="base_link" />
@@ -148,4 +143,9 @@
         <origin rpy="0 0 0" xyz="0 0 0.307" />
         <limit lower="-${PI/2}" upper="${PI/2}" effort="${effort}" velocity="${velocity}" />
+    </joint>
+    <joint name="rgb_camera_joint" type="fixed">
+        <parent link="base_link" />
+        <child link="rgb_camera" />
+        <origin xyz="0 0.45 0.2" rpy="0 -0.5 1.57"/>
     </joint>
     <joint name="joint_2" type="revolute">

Commit message: fix: camera collision

File: src/arduinobot_description/urdf/arduinobot.urdf.xacro (robot description, xacro)
@@ -36,5 +36,5 @@
         </visual>
         <collision>
-            <origin rpy="-1.1 0 0"  xyz="-0.15 0.34 0.28" />
+            <origin rpy="-${PI/2} 0 -${PI/2}" xyz="-0.1 0.125 0.15"/>
             <geometry>
                 <mesh filename="package://arduinobot_description/meshes/pi_camera.STL" scale="0.01 0.01 0.01" />
