Commit message: feat: create a new pkg - robot controller

File: src/arduinobot_description/urdf/arduinobot_gazebo.xacro (robot description, xacro)
@@ -4,12 +4,10 @@
         <xacro:if value="$(arg is_ignition)">
             <plugin filename="ign_ros2_control-system" name="ign_ros2_control::IgnitionROS2ControlPlugin">
-                <parameters>
-                </parameters>
+                <parameters>$(find arduinobot_controller)/config/arduinobot_controllers.yaml</parameters>
             </plugin>
         </xacro:if>
         <xacro:unless value="$(arg is_ignition)">
             <plugin filename="gz_ros2_control-system" name="gz_ros2_control::GazeboSimROS2ControlPlugin">
-                <parameters>
-                </parameters>
+                <parameters>$(find arduinobot_controller)/config/arduinobot_controllers.yaml</parameters>
             </plugin>
         </xacro:unless>

File: src/arduinobot_description/urdf/arduinobot_ros2_control.xacro (robot description, xacro)
@@ -1,6 +1,6 @@
 <?xml version="1.0"?>
 <robot xmlns:xacro="https://www.ros.org/wiki/xacro" name="arduinobot">
-    <xacro:property name="PI" value="3.14159" />
     <ros2_control type="system" name="RobotSystem">
+        <xacro:property name="PI" value="3.14159" />
         <xacro:if value="$(arg is_ignition)">
             <hardware>
@@ -13,36 +13,36 @@
             </hardware>
         </xacro:unless>
+        <joint name="joint_1">
+            <command_interface name="position">
+                <param name="min">-${PI / 2}</param>
+                <param name="max">${PI / 2}</param>
+            </command_interface>
+            <state_interface name="position" />
+        </joint>
+        <joint name="joint_2">
+            <command_interface name="position">
+                <param name="min">-${PI / 2}</param>
+                <param name="max">${PI / 2}</param>
+            </command_interface>
+            <state_interface name="position" />
+        </joint>
+        <joint name="joint_3">
+            <command_interface name="position">
+                <param name="min">-${PI / 2}</param>
+                <param name="max">${PI / 2}</param>
+            </command_interface>
+            <state_interface name="position" />
+        </joint>
+        <joint name="joint_4">
+            <command_interface name="position">
+                <param name="min">-${PI / 2}</param>
+                <param name="max">0.0</param>
+            </command_interface>
+            <state_interface name="position" />
+        </joint>
+        <joint name="joint_5">
+            <param name="mimic">joint_4</param>
+            <param name="multiplier">-1</param>
+        </joint>
     </ros2_control>
-    <joint name="joint_1">
-        <command_interface name="position">
-            <param name="min">-${PI / 2}</param>
-            <param name="max">${PI / 2}</param>
-        </command_interface>
-        <state_interface name="position" />
-    </joint>
-    <joint name="joint_2">
-        <command_interface name="position">
-            <param name="min">-${PI / 2}</param>
-            <param name="max">${PI / 2}</param>
-        </command_interface>
-        <state_interface name="position" />
-    </joint>
-    <joint name="joint_3">
-        <command_interface name="position">
-            <param name="min">-${PI / 2}</param>
-            <param name="max">${PI / 2}</param>
-        </command_interface>
-        <state_interface name="position" />
-    </joint>
-    <joint name="joint_4">
-        <command_interface name="position">
-            <param name="min">-${PI / 2}</param>
-            <param name="max">0.0</param>
-        </command_interface>
-        <state_interface name="position" />
-    </joint>
-    <joint name="joint_5">
-        <param name="mimic">joint_4</param>
-        <param name="multiplier">-1</param>
-    </joint>
 </robot>
